File: Fuse and Relay PCB/Fuse and Relay PCB.kicad_pcb (KiCad board)
At the start: 2 copper layers, 99 x 120 mm, 17 parts, among them J2 VCF4-1000, J3 VCF4-1000, J4 VCF4-1000, J5 VCF4-1000

Commit message: Relay Board V2 (Actual final)
Parts:
- moved C1 59.3 mm to (136.6, 153.6), turned to 180 degrees
- moved PS1 52.2 mm to (141.9, 145.4), turned to 180 degrees
- moved F5 18.6 mm to (124.0, 145.2), turned to 180 degrees
Connections:
- C1 pad 1: +12V -> Net-(J2-Pad30)
- F1 pad 1_2: (no net) -> +12V
- F1 pad 2_2: (no net) -> Net-(F1-Pad2_1)
- F2 pad 1_2: (no net) -> +12V
- F2 pad 2_2: (no net) -> Net-(F2-Pad2_1)
- F3 pad 2_2: (no net) -> Net-(F3-Pad2_1)
- F4 pad 2_2: (no net) -> Net-(F4-Pad2_1)
- F5 pad 1_2: (no net) -> Net-(PS1-+VOUT)
- F5 pad 2_2: (no net) -> Net-(F5-Pad2_1)
- MP1 pad 10: (no net) -> +12V
- MP1 pad 2: (no net) -> +12V
- MP1 pad 3: (no net) -> +12V
- MP1 pad 4: (no net) -> +12V
- MP1 pad 5: (no net) -> +12V
- MP1 pad 6: (no net) -> +12V
- MP1 pad 7: (no net) -> +12V
- MP1 pad 8: (no net) -> +12V
- MP1 pad 9: (no net) -> +12V
- PS1 pad 1: +12V -> Net-(J2-Pad30)
Routing:
- net GND: track 319.6 -> 10.6 mm
- net +12V: track 165.5 -> 0.00 mm
- net Net-(F1-Pad2_1): track 53.2 -> 0.41 mm
- net Net-(J2-Pad30): track 124.8 -> 152.0 mm
- net Net-(F2-Pad2_1): track 14.8 -> 0.28 mm
- net Net-(J5-Pad85): track 84.5 -> 70.5 mm
- net Net-(F5-Pad2_1): track 46.9 -> 34.4 mm
- net Net-(J4-Pad85): track 54.2 -> 49.1 mm
- net Net-(F4-Pad2_1): track 45.7 -> 40.9 mm
- net Net-(F3-Pad2_1): track 26.3 -> 22.9 mm
- net Net-(PS1-+VOUT): track 14.6 -> 12.1 mm
- net Net-(J3-Pad30): track 64.0 -> 62.5 mm
- net Net-(J2-Pad85): track 71.3 -> 72.6 mm
- net Net-(J4-Pad30): track 37.4 -> 36.4 mm
- added copper zone on F.Cu, net +12V
- added copper zone on B.Cu, net GND
- added copper zone on F.Cu, net Net-(F1-Pad2_1)
- added copper zone on F.Cu, net Net-(F2-Pad2_1)
Other:
- board text added: "Illini Pullers Relay Board 1/2025 Rev 2"
- board text removed: "Illini Pullers Relay Board 1/2025"
