File: Fuse and Relay PCB/Fuse and Relay PCB.kicad_sch (KiCad schematic)
At the start: 13 parts, among them J2 VCF4-1000, J3 VCF4-1000, J4 VCF4-1000, J5 VCF4-1000

Commit message: Relay Board V2 (Actual final)
Connections:
- net +12V: no longer C1.1, PS1.1 (+VIN)
- net at J2.30, Relay+5V1.6, Relay+5V1.7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: now also C1.1, PS1.1 (+VIN)
Changed lines of the file:
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@@
+	)
+	(junction
+		(at 99.06 90.17)
+		(diameter 0)
+		(color 0 0 0 0)
 	)
 	(junction
@@
 	)
 	(junction
+		(at 101.6 90.17)
+		(diameter 0)
+		(color 0 0 0 0)
+	)
+	(junction
 		(at 101.6 62.23)
 		(diameter 0)
@@
 	)
 	(junction
-		(at 101.6 90.17)
-		(diameter 0)
-		(color 0 0 0 0)
-	)
-	(junction
 		(at 99.06 102.87)
 		(diameter 0)
@@
 	)
 	(junction
-		(at 73.66 90.17)
-		(diameter 0)
-		(color 0 0 0 0)
-	)
-	(junction
 		(at 135.89 62.23)
 		(diameter 0)
@@
 	(wire
 		(pts
-			(xy 99.06 73.66) (xy 99.06 102.87)
+			(xy 99.06 73.66) (xy 99.06 90.17)
 		)
 		(stroke
@@
 	(wire
 		(pts
+			(xy 99.06 90.17) (xy 99.06 102.87)
+		)
+		(stroke
+			(width 0)
+			(type default)
+		)
+	)
+	(wire
+		(pts
 			(xy 91.44 52.07) (xy 102.87 52.07)
 		)
@@
 	(wire
 		(pts
-			(xy 73.66 90.17) (xy 101.6 90.17)
-		)
-		(stroke
-			(width 0)
-			(type default)
-		)
-	)
-	(wire
-		(pts
 			(xy 101.6 45.72) (xy 102.87 45.72)
 		)
@@
 		(pts
 			(xy 76.2 20.32) (xy 73.66 20.32)
+		)
+		(stroke
+			(width 0)
+			(type default)
+		)
+	)
+	(wire
+		(pts
+			(xy 99.06 90.17) (xy 101.6 90.17)
 		)
 		(stroke
@@
 		)
 	)
-	(text_box "1: 5V OUT\n2: J2 SIGNAL (KEYSWITCH)\n3: J3 SIGNAL\n4: J4 SIGNAL\n5: J5 SIGNAL\n6: J2 OUT\n7: J2 OUT\n8: J2 OUT\n9: J2 OUT\n10: J3 OUT\n11: J4 OUT\n12: J5 OUT"
+	(text_box "1: 5V OUT VIA J2 RELAY\n2: J2 SIGNAL (KEYSWITCH)\n3: J3 SIGNAL\n4: J4 SIGNAL\n5: J5 SIGNAL\n6: J2 OUT\n7: J2 OUT\n8: J2 OUT\n9: J2 OUT\n10: J3 OUT\n11: J4 OUT\n12: J5 OUT"
 		(exclude_from_sim no)
 		(at 218.44 90.17 0)
